Commit message: Added lidar

File: rby1_description/urdf/rby1.urdf (robot description, URDF)
Before this commit: robot rby1, 35 links, 34 joints
Links:
- added link lidar_left_link, mass 0.125; collision cylinder length=0.055 radius=0.0508; visual cylinder length=0.055 radius=0.0508
- added link lidar_right_link, mass 0.125; collision cylinder length=0.055 radius=0.0508; visual cylinder length=0.055 radius=0.0508
Joints:
- added joint lidar_left_joint: type fixed, parent base, child lidar_left_link, origin xyz=0.228 0.18 0.23 rpy=0 0 0
- added joint lidar_right_joint: type fixed, parent base, child lidar_right_link, origin xyz=0.228 -0.18 0.23 rpy=0 0 0

Commit message: lidar merging and slam mapping working

File: rby1_description/urdf/rby1.urdf (robot description, URDF)
Before this commit: robot rby1, 37 links, 36 joints
Joints:
- joint lidar_left_joint: origin xyz=0.228 0.18 0.23 rpy=0 0 0 -> xyz=0.228 0.18 0.23 rpy=0 0 0.7854
- joint lidar_right_joint: origin xyz=0.228 -0.18 0.23 rpy=0 0 0 -> xyz=0.228 -0.18 0.23 rpy=0 0 -0.7854
